Commit message: Update (Unsaved).xacro

File: testproject/(Unsaved)_description/urdf/(Unsaved).xacro (robot description, xacro)
@@ -94,5 +94,5 @@
   <parent link="base_link"/>
   <child link="right_wheel_1"/>
-  <axis xyz="0.0 -1.0 0.0"/>
+  <axis xyz="0.0 1.0 0.0"/>
 </joint>
 <joint name="Rev3" type="continuous">
